Commit message: feat(ar-mode): add AR guidance, platform parts registry, missing tables migration
- Add AR mode dashboard page and API routes
- Add parts-registry and techmedix index modules
- Add chassis/blueprints/knowledge_hub_entries/parts migration
- Update sidebar, layout, and diagnostics for AR integration
- Add fix-ollama-vision script
- Update asimov URDF model

Co-authored-by: Megan <megan@blackcatrobotics.com>

File: TechMedix-standalone/public/robots/asimov/asimov_1.urdf (robot description, URDF)
Before this commit: robot asimov_1, 26 links, 25 joints
Links:
- link left_ankle_pitch_link: geometry visual mesh filename=assets/meshes/LEFT_ANKLE_A.STL
- link left_ankle_roll_link: geometry collision sphere radius=0.005; collision sphere radius=0.005
- link left_elbow_link: geometry collision cylinder length=0.1140175425 radius=0.03; collision sphere radius=0.03
- link left_hip_pitch_link: geometry collision cylinder length=0.02 radius=0.04; collision sphere radius=0.04
- link left_hip_roll_link: geometry visual mesh filename=assets/meshes/LEFT_HIP_ROLL.STL
- link left_hip_yaw_link: geometry collision cylinder length=0.07 radius=0.04; collision sphere radius=0.04
- link left_knee_link: geometry collision cylinder length=0.18 radius=0.04; collision sphere radius=0.04
- link left_shoulder_pitch_link: geometry visual mesh filename=assets/meshes/LEFT_SHOULDER_PITCH.STL
- link left_shoulder_roll_link: geometry collision cylinder length=0.09 radius=0.035; collision sphere radius=0.035
- link left_shoulder_yaw_link: geometry visual mesh filename=assets/meshes/LEFT_SHOULDER_YAW.STL
- link left_wrist_yaw_link: geometry visual mesh filename=assets/meshes/LEFT_WRIST_YAW.STL
- link neck_pitch_link: geometry collision cylinder length=0.04 radius=0.05; collision sphere radius=0.05
- link neck_yaw_link: geometry visual mesh filename=assets/meshes/NECK_YAW.STL
- link pelvis_link: geometry collision cylinder length=0.075 radius=0.04; collision sphere radius=0.04
- link right_ankle_pitch_link: geometry visual mesh filename=assets/meshes/RIGHT_ANKLE_A.STL
- link right_ankle_roll_link: geometry collision sphere radius=0.005; collision sphere radius=0.005
- link right_elbow_link: geometry collision cylinder length=0.1140175425 radius=0.03; collision sphere radius=0.03
- link right_hip_pitch_link: geometry collision cylinder length=0.02 radius=0.04; collision sphere radius=0.04
- link right_hip_roll_link: geometry visual mesh filename=assets/meshes/RIGHT_HIP_ROLL.STL
- link right_hip_yaw_link: geometry collision cylinder length=0.07 radius=0.04; collision sphere radius=0.04
- link right_knee_link: geometry collision cylinder length=0.18 radius=0.04; collision sphere radius=0.04
- link right_shoulder_pitch_link: geometry visual mesh filename=assets/meshes/RIGHT_SHOULDER_PITCH.STL
- link right_shoulder_roll_link: geometry collision cylinder length=0.09 radius=0.035; collision sphere radius=0.035
- link right_shoulder_yaw_link: geometry visual mesh filename=assets/meshes/RIGHT_SHOULDER_YAW.STL
- link right_wrist_yaw_link: geometry visual mesh filename=assets/meshes/RIGHT_WRIST_YAW.STL
- link waist_yaw_link: geometry collision cylinder length=0.25 radius=0.06; collision sphere radius=0.06
